File: KiCad/SDISK2_ESP/SDISK2_ESP.kicad_sch (KiCad schematic)
At the start: 22 parts

Commit message: update
Parts:
- removed U?: SD_Card_Module, terence:SDCard Module, symbol terence:SD_Card_Module
- removed U?: DOIT-ESP32-DEVKIT-V1, symbol terence:DOIT-ESP32-DEVKIT-V1
- added BOARD1: ESP32DEVKITV1, ESP32-DEVKITV1, symbol terence:ESP32DEVKITV1
- added H1, H2, H3, H4: MountingHole, MountingHole:MountingHole_3mm, symbol Mechanical:MountingHole
- added J2: MicroSD, terence:MicroSD, symbol terence:MicroSD
- added LOGO1: Logo_Open_Hardware_Small, Symbol:OSHW-Symbol_6.7x6mm_SilkScreen, symbol Graphic:Logo_Open_Hardware_Small
- J1: renamed from J?; footprint Connector_IDC:IDC-Header_2x10_P2.54mm_Vertical -> Connector_IDC:IDC-Header_2x10_P2.54mm_Horizontal
- U2: renamed from U?; value SN74CB3T3245PW -> SN74CB3T3245D; footprint Package_SO:TSSOP-20_4.4x6.5mm_P0.65mm -> Package_SO:SOIC-20W_7.5x12.8mm_P1.27mm
- U5: renamed from U?; value 74HC125 -> 74HC125D; footprint Package_DIP:DIP-14_W7.62mm -> Package_SO:SOIC-14_3.9x8.7mm_P1.27mm
- U8: renamed from U?; footprint terence:0.96OLED I2C -> terence:1.3 OLED I2C
- gave numbers to parts that had none: 12
Connections:
- net W_REQUEST_L is gone; now on net xW_REQUEST: R3.2
- net +5V: now also BOARD1.VIN
- net BT_DOWN: now also BOARD1.D16
- net BT_ENTER: now also BOARD1.D17
- net BT_UP: now also BOARD1.D15
- net DRIVE_EN: now also U2.8 (A6)
- net GND: now also BOARD1.GND, BOARD1.GND@1, J2.6 (VSS)
- net SCL: now also BOARD1.D22
- net SDA: now also BOARD1.D21
- net SD_CLK/CLK: now also BOARD1.D18, J2.5 (CLK)
- net SD_CS/CS: now also BOARD1.D5, J2.2 (DAT3/CD)
- net SD_DI/MOSI: now also BOARD1.D23, J2.3 (CMD)
- net SD_DO/MISO: now also BOARD1.D19, J2.7 (DAT0)
- net STEP 0: now also U2.3 (A1)
- net STEP 1: now also U2.4 (A2)
- net STEP 2: now also U2.5 (A3)
- net STEP 3: now also U2.6 (A4)
- net VCC: now also BOARD1.3V3, J2.4 (VDD)
- net WRITE: now also U2.7 (A5)
- net W_REQUEST: now also U2.9 (A7)
- net at U5.2: now also BOARD1.D14
- net at R1.1: now also BOARD1.D13
- net xW_REQUEST: now reaches U2.11 (B7)
- net xW_REQUEST: now also BOARD1.D27
- net xDRIVE_EN: now reaches U2.12 (B6)
- net xDRIVE_EN: now also BOARD1.D26
- net xWRITE: now reaches U2.13 (B5)
- net xWRITE: now also BOARD1.D25
- net xSTEP 3: now reaches U2.14 (B4)
- net xSTEP 3: now also BOARD1.D33
- net xSTEP 2: now reaches U2.15 (B3)
- net xSTEP 2: now also BOARD1.D32
- net xSTEP 1: now reaches U2.16 (B2)
- net xSTEP 1: now also BOARD1.D35
- net xSTEP 0: now reaches U2.17 (B1)
- net xSTEP 0: now also BOARD1.D34
- net at U5.5: now also BOARD1.D12
- net SD_Eject renamed Card_Detect
- net Card_Detect: now also BOARD1.D2, J2.9 (Card_Detect)
- no-connect marks 12 -> 20
Other:
- moved on the sheet: C1, C2, C3, D1, R1, R2, R3, R4, R5, U2, U5A, U5B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
